File: sch/LightStick/LightStick.kicad_pcb (KiCad board)
At the start: 2 copper layers, 25 x 73 mm, 19 parts, among them J1 +BATT, J2 GND, Q1 IRLML0030, Q2 IRLML0030, Q3 IRLML0030, Q4 IRLML0030, SW1 SW_Push, SW2 SW_Push, U2 XIAO-nRF54l15-SMD

Commit message: Raytac Module version
Parts:
- removed JP1: LiPo?, Jumper:SolderJumper-3_P1.3mm_Bridged12_RoundedPad1.0x1.5mm
- removed U2: XIAO-nRF54l15-SMD, parts:XIAO-nRF54l15-SMD
- added J3: SWD, Connector_JST:JST_SH_SM05B-SRSS-TB_1x05-1MP_P1.00mm_Horizontal, B.Cu at (195.8, 138.7)
- added J4: MIC, Connector_JST:JST_SH_SM04B-SRSS-TB_1x04-1MP_P1.00mm_Horizontal, B.Cu at (186.6, 138.7)
- added J5: USB_C_Receptacle_USB2.0_14P, Connector_USB:USB_C_Receptacle_Palconn_UTC16-G, F.Cu at (186.6, 137.7)
- added R1: 5.1k, Resistor_SMD:R_0603_1608Metric_Pad0.98x0.95mm_HandSolder, F.Cu at (184.8, 132.2)
- added R2: 5.1k, Resistor_SMD:R_0603_1608Metric_Pad0.98x0.95mm_HandSolder, F.Cu at (190.0, 132.4)
- added R3: 33, Resistor_SMD:R_0603_1608Metric_Pad0.98x0.95mm_HandSolder, F.Cu at (187.8, 128.5)
- added R4: 33, Resistor_SMD:R_0603_1608Metric_Pad0.98x0.95mm_HandSolder, F.Cu at (189.6, 128.5)
- added U1: MDBT50Q-1MV2, RF_Module:Raytac_MDBT50Q, B.Cu at (192.7, 128.9)
- J1, J2: moved to F.Cu
- moved J2 12.7 mm to (182.2, 124.4), turned to 0 degrees
- moved J1 7.88 mm to (199.1, 120.8), turned to 0 degrees
Routing:
- net VBUS: track 0.00 -> 19.4 mm, vias 0 -> 1
- net /RST: track 0.00 -> 15.6 mm, vias 0 -> 2
- net Net-(JP1-B): track 15.5 -> 0.00 mm, vias 1 -> 0
- net Net-(J3-Pin_3): track 0.00 -> 15.4 mm, vias 0 -> 2
- net Net-(J3-Pin_4): track 0.00 -> 15.2 mm, vias 0 -> 2
- net +BATT: track 32.5 -> 44.4 mm, vias 0 -> 3
- net Net-(J5-D+-PadA6): track 0.00 -> 9.33 mm
- net /PDM_CLK: track 0.00 -> 9.21 mm
- net Net-(J5-D--PadA7): track 0.00 -> 7.94 mm
- net /PDM_DATA: track 0.00 -> 7.81 mm
- net +3.3V: track 43.4 -> 36.7 mm, vias 2 -> 1
- net /SW1: track 17.0 -> 11.0 mm, vias 1 -> 2
- net Net-(JP1-A): track 4.64 -> 0.00 mm, vias 1 -> 0
- net /D+: track 0.00 -> 4.32 mm, vias 0 -> 1
- net /D-: track 0.00 -> 3.89 mm, vias 0 -> 1
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Other:
- board size 25 x 73 mm -> 25 x 71.5 mm

Commit message: wip
Parts:
- removed D1: LED_RGBW, parts:XL-5050RGBW
Routing:
- net Net-(D1-WA): track 22.3 -> 5.02 mm
- net /LED_R: track 21.5 -> 4.72 mm
- net Net-(D1-BA): track 19.5 -> 5.88 mm
- net /LED_G: track 20.6 -> 7.26 mm
- net /LED_B: track 19.2 -> 9.77 mm
- net Net-(D1-GA): track 15.9 -> 6.62 mm
- net /LED_W: track 17.1 -> 11.6 mm
- net Net-(D1-RA): track 12.6 -> 7.19 mm
- removed copper zone on F.Cu, net Net-(D1-BA)
- removed copper zone on F.Cu, net Net-(D1-GA)
- removed copper zone on F.Cu, net Net-(D1-RA)
- removed copper zone on F.Cu, net Net-(D1-WA)
Other:
- board size 25 x 71.5 mm -> 23 x 36.5 mm
